File: phoenix/phoenix.sch (KiCad schematic (older format))
At the start: 28 parts, among them J1 Ultrafit_2, J2 Micro_SD_Card_Det, P1 CONN_02X03, U1 ATMEGA328P-AU, U2 SI4838DY, U3 MMA8451QT, U4 L6932D1.2, Y1 Crystal_SMD

Commit message: Started layout
Parts:
- BT1: footprint (none) -> rocketry:battery_holder
- C1, C2, C3, C4, C5, C6, C7: footprint footprints:C_0805_OEM -> rocketry:C_0805_OEM
- D1, D2, D3: footprint footprints:LED_0805_OEM -> rocketry:LED_0805_OEM
- J1: footprint footprints:Ultrafit_2 -> rocketry:Ultrafit_2_RA
- J2: footprint (none) -> rocketry:SD-Card
- P1: footprint footprints:Pin_Header_Straight_2x03 -> rocketry:Pin_Header_Straight_2x03
- R1, R4, R5, R6, R7, R8, R9: footprint footprints:R_0805_OEM -> rocketry:R_0805_OEM
- R2, R3: footprint (none) -> rocketry:R_0805_OEM
- U2: footprint (none) -> rocketry:IRLML6344TRPBFCT-ND
- U3: footprint footprints:MMA8451QT -> rocketry:MMA8451QT
- U4: footprint footprints:L6932D1.2TR -> rocketry:L6932D1.2TR
- Y1: footprint footprints:Crystal_SMD_FA238 -> rocketry:Crystal_SMD_FA238
Changed lines of the file:
@@
 F 0 "BT1" V 17850 6450 50  0000 L CNN
 F 1 "3.7V Lipo" V 17500 6300 50  0000 L CNN
-F 2 "" V 17700 6510 50  0001 C CNN
+F 2 "rocketry:battery_holder" V 17700 6510 50  0001 C CNN
 F 3 "" V 17700 6510 50  0001 C CNN
 	1    17700 6450
@@
 F 0 "J2" H 19200 6450 50  0000 C CNN
 F 1 "Micro_SD_Card_Det" H 20500 6450 50  0000 R CNN
-F 2 "" H 21900 6450 50  0001 C CNN
+F 2 "rocketry:SD-Card" H 21900 6450 50  0001 C CNN
 F 3 "" H 19850 5850 50  0001 C CNN
 	1    19850 5750
@@
 F 0 "R7" V 18080 1650 50  0000 C CNN
 F 1 "R_100" V 17900 1650 50  0000 C CNN
-F 2 "footprints:R_0805_OEM" H 17930 1650 50  0001 C CNN
+F 2 "rocketry:R_0805_OEM" H 17930 1650 50  0001 C CNN
 F 3 "https://www.seielect.com/Catalog/SEI-rncp.pdf" H 18080 1650 50  0001 C CNN
 F 4 "Digi-Key" H 18000 1650 60  0001 C CNN "MFN"
@@
 F 0 "C5" H 17850 2100 50  0000 L CNN
 F 1 "C_100pF" H 17650 1900 50  0000 L CNN
-F 2 "footprints:C_0805_OEM" H 18038 1850 50  0001 C CNN
+F 2 "rocketry:C_0805_OEM" H 18038 1850 50  0001 C CNN
 F 3 "https://content.kemet.com/datasheets/KEM_C1003_C0G_SMD.pdf" H 18025 2100 50  0001 C CNN
 F 4 "399-1122-1-ND" H 18000 2000 60  0001 C CNN "MPN"
@@
 F 0 "P1" H 17150 5800 50  0000 C CNN
 F 1 "CONN_02X03" H 17150 5400 50  0000 C CNN
-F 2 "footprints:Pin_Header_Straight_2x03" H 17150 4400 50  0001 C CNN
+F 2 "rocketry:Pin_Header_Straight_2x03" H 17150 4400 50  0001 C CNN
 F 3 "http://portal.fciconnect.com/Comergent//fci/drawing/67996.pdf" H 17150 4400 50  0001 C CNN
 F 4 "609-3234-ND" H 17150 5600 60  0001 C CNN "MPN"
@@
 F 0 "R9" V 20580 2750 50  0000 C CNN
 F 1 "R_10k" V 20400 2750 50  0000 C CNN
-F 2 "footprints:R_0805_OEM" H 20430 2750 50  0001 C CNN
+F 2 "rocketry:R_0805_OEM" H 20430 2750 50  0001 C CNN
 F 3 "http://www.bourns.com/data/global/pdfs/CRS.pdf" H 20580 2750 50  0001 C CNN
 F 4 "CRS0805-FX-1002ELFCT-ND" H 20500 2750 60  0001 C CNN "MPN"
@@
 F 0 "D2" H 15750 5100 50  0000 C CNN
 F 1 "LED_0805" H 15700 5300 50  0000 C CNN
-F 2 "footprints:LED_0805_OEM" H 15650 5200 50  0001 C CNN
+F 2 "rocketry:LED_0805_OEM" H 15650 5200 50  0001 C CNN
 F 3 "http://www.osram-os.com/Graphics/XPic9/00078860_0.pdf" H 15750 5300 50  0001 C CNN
 F 4 "475-1410-1-ND" H 15750 5200 60  0001 C CNN "MPN"
@@
 F 0 "R5" V 15830 5650 50  0000 C CNN
 F 1 "R_200" V 15650 5650 50  0000 C CNN
-F 2 "footprints:R_0805_OEM" H 15680 5650 50  0001 C CNN
+F 2 "rocketry:R_0805_OEM" H 15680 5650 50  0001 C CNN
 F 3 "https://www.seielect.com/Catalog/SEI-RMCF_RMCP.pdf" H 15830 5650 50  0001 C CNN
 F 4 "Digi-Key" H 15750 5650 60  0001 C CNN "MFN"
@@
 F 0 "D3" H 16100 5100 50  0000 C CNN
 F 1 "LED_0805" H 16050 5300 50  0000 C CNN
-F 2 "footprints:LED_0805_OEM" H 16000 5200 50  0001 C CNN
+F 2 "rocketry:LED_0805_OEM" H 16000 5200 50  0001 C CNN
 F 3 "http://www.osram-os.com/Graphics/XPic9/00078860_0.pdf" H 16100 5300 50  0001 C CNN
 F 4 "475-1410-1-ND" H 16100 5200 60  0001 C CNN "MPN"
@@
 F 0 "R6" V 16180 5650 50  0000 C CNN
 F 1 "R_200" V 16000 5650 50  0000 C CNN
-F 2 "footprints:R_0805_OEM" H 16030 5650 50  0001 C CNN
+F 2 "rocketry:R_0805_OEM" H 16030 5650 50  0001 C CNN
 F 3 "https://www.seielect.com/Catalog/SEI-RMCF_RMCP.pdf" H 16180 5650 50  0001 C CNN
 F 4 "Digi-Key" H 16100 5650 60  0001 C CNN "MFN"
@@
 F 0 "D1" H 15400 5100 50  0000 C CNN
 F 1 "LED_0805" H 15350 5300 50  0000 C CNN
-F 2 "footprints:LED_0805_OEM" H 15300 5200 50  0001 C CNN
+F 2 "rocketry:LED_0805_OEM" H 15300 5200 50  0001 C CNN
 F 3 "http://www.osram-os.com/Graphics/XPic9/00078860_0.pdf" H 15400 5300 50  0001 C CNN
 F 4 "475-1410-1-ND" H 15400 5200 60  0001 C CNN "MPN"
@@
 F 0 "R4" V 15480 5650 50  0000 C CNN
 F 1 "R_200" V 15300 5650 50  0000 C CNN
-F 2 "footprints:R_0805_OEM" H 15330 5650 50  0001 C CNN
+F 2 "rocketry:R_0805_OEM" H 15330 5650 50  0001 C CNN
 F 3 "https://www.seielect.com/Catalog/SEI-RMCF_RMCP.pdf" H 15480 5650 50  0001 C CNN
 F 4 "Digi-Key" H 15400 5650 60  0001 C CNN "MFN"
@@
 F 0 "J1" H 6900 1550 60  0000 C CNN
 F 1 "Ultrafit_2" H 7000 1200 60  0000 C CNN
-F 2 "footprints:Ultrafit_2" H 6800 1450 60  0001 C CNN
+F 2 "rocketry:Ultrafit_2_RA" H 6800 1450 60  0001 C CNN
 F 3 "" H 6900 1550 60  0001 C CNN
 F 4 "https://www.digikey.com/product-detail/en/molex-llc/1722861102/WM11570-ND/5344267" H 7000 1650 60  0001 C CNN "PurchasingLink"
@@
 F 0 "U3" H 11750 4650 60  0000 C CNN
 F 1 "MMA8451QT" H 11750 4500 60  0000 C CNN
-F 2 "footprints:MMA8451QT" H 11750 5540 60  0001 C CNN
+F 2 "rocketry:MMA8451QT" H 11750 5540 60  0001 C CNN
 F 3 "" H 10550 5300 60  0000 C CNN
 F 4 "https://www.digikey.com/products/en?mpart=MMA8451QT&v=568" H 11850 5800 60  0001 C CNN "PurchasingLinks"
@@
 F 0 "C1" H 9825 5800 50  0000 L CNN
 F 1 "C_0.1uF" H 9800 5550 50  0000 L CNN
-F 2 "footprints:C_0805_OEM" H 9838 5550 50  0001 C CNN
+F 2 "rocketry:C_0805_OEM" H 9838 5550 50  0001 C CNN
 F 3 "http://datasheets.avx.com/X7RDielectric.pdf" H 9825 5800 50  0001 C CNN
 F 4 "478-3352-1-ND" H 9800 5700 60  0001 C CNN "MPN"
@@
 F 0 "R1" V 10280 5750 50  0000 C CNN
 F 1 "R_10k" V 10100 5750 50  0000 C CNN
-F 2 "footprints:R_0805_OEM" H 10130 5750 50  0001 C CNN
+F 2 "rocketry:R_0805_OEM" H 10130 5750 50  0001 C CNN
 F 3 "http://www.bourns.com/data/global/pdfs/CRS.pdf" H 10280 5750 50  0001 C CNN
 F 4 "CRS0805-FX-1002ELFCT-ND" H 10200 5750 60  0001 C CNN "MPN"
@@
 F 0 "C2" H 9325 5800 50  0000 L CNN
 F 1 "C_0.1uF" H 9325 5600 50  0000 L CNN
-F 2 "footprints:C_0805_OEM" H 9338 5550 50  0001 C CNN
+F 2 "rocketry:C_0805_OEM" H 9338 5550 50  0001 C CNN
 F 3 "http://datasheets.avx.com/X7RDielectric.pdf" H 9325 5800 50  0001 C CNN
 F 4 "478-3352-1-ND" H 9300 5700 60  0001 C CNN "MPN"
@@
 F 0 "U4" H 12150 2550 60  0000 C CNN
 F 1 "L6932D1.2" H 12150 2450 60  0000 C CNN
-F 2 "footprints:L6932D1.2TR" H 12150 2390 60  0001 C CNN
+F 2 "rocketry:L6932D1.2TR" H 12150 2390 60  0001 C CNN
 F 3 "" H 12150 2550 60  0000 C CNN
 F 4 "https://www.digikey.com/product-detail/en/stmicroelectronics/L6932D1.2TR/497-5724-1-ND/1299970" H 12250 2650 60  0001 C CNN "purchasingLink"
@@
 F 0 "C4" H 10225 2350 50  0000 L CNN
 F 1 "C_10uF" H 10225 2150 50  0000 L CNN
-F 2 "footprints:C_0805_OEM" H 10238 2100 50  0001 C CNN
+F 2 "rocketry:C_0805_OEM" H 10238 2100 50  0001 C CNN
 F 3 "http://datasheets.avx.com/cx5r.pdf" H 10225 2350 50  0001 C CNN
 F 4 "478-5167-1-ND" H 10200 2250 60  0001 C CNN "MPN"
@@
 F 0 "R3" V 10680 2550 50  0000 C CNN
 F 1 "5K" V 10600 2550 50  0000 C CNN
-F 2 "" V 10530 2550 50  0001 C CNN
+F 2 "rocketry:R_0805_OEM" V 10530 2550 50  0001 C CNN
 F 3 "" H 10600 2550 50  0001 C CNN
 	1    10600 2550
@@
 F 0 "R2" V 10680 2150 50  0000 C CNN
 F 1 "9K" V 10600 2150 50  0000 C CNN
-F 2 "" V 10530 2150 50  0001 C CNN
+F 2 "rocketry:R_0805_OEM" V 10530 2150 50  0001 C CNN
 F 3 "" H 10600 2150 50  0001 C CNN
 	1    10600 2150
@@
 F 0 "C3" H 9825 2350 50  0000 L CNN
 F 1 "C_10uF" H 9825 2150 50  0000 L CNN
-F 2 "footprints:C_0805_OEM" H 9838 2100 50  0001 C CNN
+F 2 "rocketry:C_0805_OEM" H 9838 2100 50  0001 C CNN
 F 3 "http://datasheets.avx.com/cx5r.pdf" H 9825 2350 50  0001 C CNN
 F 4 "478-5167-1-ND" H 9800 2250 60  0001 C CNN "MPN"
@@
 F 0 "U2" H 6150 2300 60  0000 C CNN
 F 1 "SI4838DY" H 6150 2000 60  0000 C CNN
-F 2 "" H 6150 2150 60  0001 C CNN
+F 2 "rocketry:IRLML6344TRPBFCT-ND" H 6150 2150 60  0001 C CNN
 F 3 "" H 6150 2300 60  0001 C CNN
 F 4 "https://www.digikey.com/product-detail/en/vishay-siliconix/SI4838DY-T1-E3/SI4838DY-T1-E3TR-ND/1656477" H 6250 2400 60  0001 C CNN "purchasingLinks"
@@
 F 0 "R8" V 20430 3950 50  0000 C CNN
 F 1 "R_10k" V 20250 3950 50  0000 C CNN
-F 2 "footprints:R_0805_OEM" H 20280 3950 50  0001 C CNN
+F 2 "rocketry:R_0805_OEM" H 20280 3950 50  0001 C CNN
 F 3 "http://www.bourns.com/data/global/pdfs/CRS.pdf" H 20430 3950 50  0001 C CNN
 F 4 "CRS0805-FX-1002ELFCT-ND" H 20350 3950 60  0001 C CNN "MPN"
@@
 F 0 "Y1" H 21700 2175 50  0000 L CNN
 F 1 "Crystal_SMD" H 21300 2300 50  0000 L CNN
-F 2 "footprints:Crystal_SMD_FA238" H 21600 2075 50  0001 C CNN
+F 2 "rocketry:Crystal_SMD_FA238" H 21600 2075 50  0001 C CNN
 F 3 "https://support.epson.biz/td/api/doc_check.php?dl=brief_FA-238V_en.pdf" H 21700 2175 50  0001 C CNN
 F 4 "Digi-Key" H 21650 2000 60  0001 C CNN "MFN"
@@
 F 0 "C6" H 21425 2250 50  0000 L CNN
 F 1 "C_30pF" H 21425 2050 50  0000 L CNN
-F 2 "footprints:C_0805_OEM" H 21438 2000 50  0001 C CNN
+F 2 "rocketry:C_0805_OEM" H 21438 2000 50  0001 C CNN
 F 3 "https://media.digikey.com/pdf/Data%20Sheets/Samsung%20PDFs/CL_Series_MLCC_ds.pdf" H 21425 2250 50  0001 C CNN
 F 4 "1276-1130-1-ND" H 21400 2150 60  0001 C CNN "MPN"
@@
 F 0 "C7" H 21925 2250 50  0000 L CNN
 F 1 "C_30pF" H 21925 2050 50  0000 L CNN
-F 2 "footprints:C_0805_OEM" H 21938 2000 50  0001 C CNN
+F 2 "rocketry:C_0805_OEM" H 21938 2000 50  0001 C CNN
 F 3 "https://media.digikey.com/pdf/Data%20Sheets/Samsung%20PDFs/CL_Series_MLCC_ds.pdf" H 21925 2250 50  0001 C CNN
 F 4 "1276-1130-1-ND" H 21900 2150 60  0001 C CNN "MPN"

Commit message: fixed power transistor. Added to layout
Parts:
- removed U2: SI4838DY, rocketry:IRLML6344TRPBFCT-ND, symbol SI4838DY
- added Q1: IRLML6344, rocketry:IRLML6344TRPBFCT-ND, symbol IRLML6344
Connections:
- wire segments 46 -> 42
Other:
- moved on the sheet: C3, C4, J1, R2, R3, U4
Changed lines of the file:
@@
 EESchema Schematic File Version 2
+LIBS:power
+LIBS:device
+LIBS:switches
+LIBS:relays
+LIBS:motors
+LIBS:transistors
+LIBS:conn
+LIBS:linear
+LIBS:regul
+LIBS:74xx
+LIBS:cmos4000
+LIBS:adc-dac
+LIBS:memory
+LIBS:xilinx
+LIBS:microcontrollers
+LIBS:dsp
+LIBS:microchip
+LIBS:analog_switches
+LIBS:motorola
+LIBS:texas
+LIBS:intel
+LIBS:audio
+LIBS:interface
+LIBS:digital-audio
+LIBS:philips
+LIBS:display
+LIBS:cypress
+LIBS:siliconi
+LIBS:opto
+LIBS:atmel
+LIBS:contrib
+LIBS:valves
 LIBS:rocketry
 LIBS:phoenix-cache
@@
 L Ultrafit_2 J1
 U 1 1 5ABC44C9
-P 6900 1400
-F 0 "J1" H 6900 1550 60  0000 C CNN
-F 1 "Ultrafit_2" H 7000 1200 60  0000 C CNN
-F 2 "rocketry:Ultrafit_2_RA" H 6800 1450 60  0001 C CNN
-F 3 "" H 6900 1550 60  0001 C CNN
-F 4 "https://www.digikey.com/product-detail/en/molex-llc/1722861102/WM11570-ND/5344267" H 7000 1650 60  0001 C CNN "PurchasingLink"
-F 5 "Digi-Key" H 7100 1750 60  0001 C CNN "MFN"
-F 6 "WM11570-ND" H 7200 1850 60  0001 C CNN "MPN"
-F 7 "Value" H 7300 1950 60  0001 C CNN "Package"
-	1    6900 1400
+P 9550 1850
+F 0 "J1" H 9550 2000 60  0000 C CNN
+F 1 "Ultrafit_2" H 9650 1650 60  0000 C CNN
+F 2 "rocketry:Ultrafit_2_RA" H 9450 1900 60  0001 C CNN
+F 3 "" H 9550 2000 60  0001 C CNN
+F 4 "https://www.digikey.com/product-detail/en/molex-llc/1722861102/WM11570-ND/5344267" H 9650 2100 60  0001 C CNN "PurchasingLink"
+F 5 "Digi-Key" H 9750 2200 60  0001 C CNN "MFN"
+F 6 "WM11570-ND" H 9850 2300 60  0001 C CNN "MPN"
+F 7 "Value" H 9950 2400 60  0001 C CNN "Package"
+	1    9550 1850
 	1    0    0    -1
 $EndComp
@@
 L L6932D1.2 U4
 U 1 1 5AC43804
-P 11050 2150
-F 0 "U4" H 12150 2550 60  0000 C CNN
-F 1 "L6932D1.2" H 12150 2450 60  0000 C CNN
-F 2 "rocketry:L6932D1.2TR" H 12150 2390 60  0001 C CNN
-F 3 "" H 12150 2550 60  0000 C CNN
-F 4 "https://www.digikey.com/product-detail/en/stmicroelectronics/L6932D1.2TR/497-5724-1-ND/1299970" H 12250 2650 60  0001 C CNN "purchasingLink"
-	1    11050 2150
+P 12650 2150
+F 0 "U4" H 13750 2550 60  0000 C CNN
+F 1 "L6932D1.2" H 13750 2450 60  0000 C CNN
+F 2 "rocketry:L6932D1.2TR" H 13750 2390 60  0001 C CNN
+F 3 "" H 13750 2550 60  0000 C CNN
+F 4 "https://www.digikey.com/product-detail/en/stmicroelectronics/L6932D1.2TR/497-5724-1-ND/1299970" H 13850 2650 60  0001 C CNN "purchasingLink"
+	1    12650 2150
 	1    0    0    -1
 $EndComp
@@
 L C_10uF C4
 U 1 1 5AC43E21
-P 10200 2250
-F 0 "C4" H 10225 2350 50  0000 L CNN
-F 1 "C_10uF" H 10225 2150 50  0000 L CNN
-F 2 "rocketry:C_0805_OEM" H 10238 2100 50  0001 C CNN
-F 3 "http://datasheets.avx.com/cx5r.pdf" H 10225 2350 50  0001 C CNN
-F 4 "478-5167-1-ND" H 10200 2250 60  0001 C CNN "MPN"
-F 5 "Digi-Key" H 10200 2250 60  0001 C CNN "MFN"
-F 6 "Value" H 10200 2250 60  0001 C CNN "Package"
-F 7 "https://www.digikey.com/product-detail/en/avx-corporation/0805ZD106KAT2A/478-5167-1-ND/1913257" H 10625 2750 60  0001 C CNN "PurchasingLink"
-	1    10200 2250
-	1    0    0    -1
-$EndComp
-Text Label 10200 2100 1    60   ~ 0
+P 11800 2250
+F 0 "C4" H 11825 2350 50  0000 L CNN
+F 1 "C_10uF" H 11825 2150 50  0000 L CNN
+F 2 "rocketry:C_0805_OEM" H 11838 2100 50  0001 C CNN
+F 3 "http://datasheets.avx.com/cx5r.pdf" H 11825 2350 50  0001 C CNN
+F 4 "478-5167-1-ND" H 11800 2250 60  0001 C CNN "MPN"
+F 5 "Digi-Key" H 11800 2250 60  0001 C CNN "MFN"
+F 6 "Value" H 11800 2250 60  0001 C CNN "Package"
+F 7 "https://www.digikey.com/product-detail/en/avx-corporation/0805ZD106KAT2A/478-5167-1-ND/1913257" H 12225 2750 60  0001 C CNN "PurchasingLink"
+	1    11800 2250
+	1    0    0    -1
+$EndComp
+Text Label 11800 2100 1    60   ~ 0
 VIN
 $Comp
 L 5K R3
 U 1 1 5AC3FF90
-P 10600 2550
-F 0 "R3" V 10680 2550 50  0000 C CNN
-F 1 "5K" V 10600 2550 50  0000 C CNN
-F 2 "rocketry:R_0805_OEM" V 10530 2550 50  0001 C CNN
-F 3 "" H 10600 2550 50  0001 C CNN
-	1    10600 2550
+P 12200 2550
+F 0 "R3" V 12280 2550 50  0000 C CNN
+F 1 "5K" V 12200 2550 50  0000 C CNN
+F 2 "rocketry:R_0805_OEM" V 12130 2550 50  0001 C CNN
+F 3 "" H 12200 2550 50  0001 C CNN
+	1    12200 2550
 	1    0    0    -1
 $EndComp
@@
 L 5K R2
 U 1 1 5AC404C1
-P 10600 2150
-F 0 "R2" V 10680 2150 50  0000 C CNN
-F 1 "9K" V 10600 2150 50  0000 C CNN
-F 2 "rocketry:R_0805_OEM" V 10530 2150 50  0001 C CNN
-F 3 "" H 10600 2150 50  0001 C CNN
-	1    10600 2150
-	1    0    0    -1
-$EndComp
-Text Label 10600 2700 3    60   ~ 0
-GND
-Text Label 11050 2250 2    60   ~ 0
+P 12200 2150
+F 0 "R2" V 12280 2150 50  0000 C CNN
+F 1 "9K" V 12200 2150 50  0000 C CNN
+F 2 "rocketry:R_0805_OEM" V 12130 2150 50  0001 C CNN
+F 3 "" H 12200 2150 50  0001 C CNN
+	1    12200 2150
+	1    0    0    -1
+$EndComp
+Text Label 12200 2700 3    60   ~ 0
+GND
+Text Label 12650 2250 2    60   ~ 0
 VIN
-Text Label 11050 2150 2    60   ~ 0
+Text Label 12650 2150 2    60   ~ 0
 VIN
 $Comp
 L C_10uF C3
 U 1 1 5AC40A51
-P 9800 2250
-F 0 "C3" H 9825 2350 50  0000 L CNN
-F 1 "C_10uF" H 9825 2150 50  0000 L CNN
-F 2 "rocketry:C_0805_OEM" H 9838 2100 50  0001 C CNN
-F 3 "http://datasheets.avx.com/cx5r.pdf" H 9825 2350 50  0001 C CNN
-F 4 "478-5167-1-ND" H 9800 2250 60  0001 C CNN "MPN"
-F 5 "Digi-Key" H 9800 2250 60  0001 C CNN "MFN"
-F 6 "Value" H 9800 2250 60  0001 C CNN "Package"
-F 7 "https://www.digikey.com/product-detail/en/avx-corporation/0805ZD106KAT2A/478-5167-1-ND/1913257" H 10225 2750 60  0001 C CNN "PurchasingLink"
-	1    9800 2250
+P 11400 2250
+F 0 "C3" H 11425 2350 50  0000 L CNN
+F 1 "C_10uF" H 11425 2150 50  0000 L CNN
+F 2 "rocketry:C_0805_OEM" H 11438 2100 50  0001 C CNN
+F 3 "http://datasheets.avx.com/cx5r.pdf" H 11425 2350 50  0001 C CNN
+F 4 "478-5167-1-ND" H 11400 2250 60  0001 C CNN "MPN"
+F 5 "Digi-Key" H 11400 2250 60  0001 C CNN "MFN"
+F 6 "Value" H 11400 2250 60  0001 C CNN "Package"
+F 7 "https://www.digikey.com/product-detail/en/avx-corporation/0805ZD106KAT2A/478-5167-1-ND/1913257" H 11825 2750 60  0001 C CNN "PurchasingLink"
+	1    11400 2250
 	1    0    0    -1
 $EndComp
@@
 	10200 5900 10550 5900
 Wire Wire Line
-	10600 2300 10600 2400
-Connection ~ 10600 2350
-Wire Wire Line
-	10600 2350 11050 2350
-Wire Wire Line
-	13250 2150 13250 2450
-Connection ~ 13250 2250
-Connection ~ 13250 2350
-Wire Wire Line
-	13250 2250 13350 2250
-Text Label 13350 2250 0    60   ~ 0
-GND
-Text Label 9800 2400 3    60   ~ 0
-GND
-$Comp
-L SI4838DY U2
-U 1 1 5AC427B1
-P 6150 2150
-F 0 "U2" H 6150 2300 60  0000 C CNN
-F 1 "SI4838DY" H 6150 2000 60  0000 C CNN
-F 2 "rocketry:IRLML6344TRPBFCT-ND" H 6150 2150 60  0001 C CNN
-F 3 "" H 6150 2300 60  0001 C CNN
-F 4 "https://www.digikey.com/product-detail/en/vishay-siliconix/SI4838DY-T1-E3/SI4838DY-T1-E3TR-ND/1656477" H 6250 2400 60  0001 C CNN "purchasingLinks"
-	1    6150 2150
-	1    0    0    -1
-$EndComp
-Wire Wire Line
-	5550 2000 5550 2200
-Connection ~ 5550 2100
-Wire Wire Line
-	5550 2100 5400 2100
-Wire Wire Line
-	6750 2000 6750 2300
-Connection ~ 6750 2100
-Wire Wire Line
-	6750 2100 7250 2100
+	12200 2300 12200 2400
+Connection ~ 12200 2350
+Wire Wire Line
+	12200 2350 12650 2350
+Wire Wire Line
+	14850 2150 14850 2450
+Connection ~ 14850 2250
+Connection ~ 14850 2350
+Wire Wire Line
+	14850 2250 14950 2250
+Text Label 14950 2250 0    60   ~ 0
+GND
+Text Label 11400 2400 3    60   ~ 0
+GND
 Text Label 20550 3800 0    60   ~ 0
 SEPERATE
@@
 GND
 Connection ~ 20350 3800
-Text Label 5550 2300 2    60   ~ 0
+Text Label 9600 2450 2    60   ~ 0
 SEPERATE
-Text Label 5400 2100 2    60   ~ 0
+Text Label 9900 2650 3    60   ~ 0
 GND
 Text Notes 10650 4750 0    60   ~ 0
 Accelerometer
-Text Notes 11400 1600 0    60   ~ 0
+Text Notes 13000 1600 0    60   ~ 0
 Linear Regulator\n
-Text Notes 5700 1750 0    60   ~ 0
+Text Notes 8350 2200 0    60   ~ 0
 N-Channel Transistor\n
 $Comp
@@
 Connection ~ 21650 2300
 Wire Wire Line
-	7250 2100 7250 1450
-Wire Wire Line
-	7250 1450 7150 1450
-Connection ~ 6750 2200
+	9900 1900 9800 1900
 NoConn ~ 18300 2950
 NoConn ~ 18300 2850
@@
 	9800 5450 9800 5550
 Connection ~ 10200 5450
-Text Label 10200 2400 3    60   ~ 0
-GND
-Text Label 7150 1350 0    60   ~ 0
-3.3V
-Text Label 10600 2000 2    60   ~ 0
-3.3V
-Text Label 11050 2450 2    60   ~ 0
-3.3V
-Text Label 9800 2100 2    60   ~ 0
+Text Label 11800 2400 3    60   ~ 0
+GND
+Text Label 9800 1800 0    60   ~ 0
+3.3V
+Text Label 12200 2000 2    60   ~ 0
+3.3V
+Text Label 12650 2450 2    60   ~ 0
+3.3V
+Text Label 11400 2100 2    60   ~ 0
 3.3V
 Text Label 20500 2600 0    60   ~ 0
 3.3V
 NoConn ~ 20650 6250
+$Comp
+L IRLML6344 Q1
+U 1 1 5ACFF80D
+P 9800 2450
+F 0 "Q1" H 10000 2525 50  0000 L CNN
+F 1 "IRLML6344" H 10000 2450 50  0001 L CNN
+F 2 "rocketry:IRLML6344TRPBFCT-ND" H 10000 2375 50  0001 L CIN
+F 3 "https://www.infineon.com/dgdl/irlml6344pbf.pdf?fileId=5546d462533600a4015356689c44262c" H 10000 2525 50  0001 L CNN
+F 4 "https://www.digikey.com/product-detail/en/infineon-technologies/IRLML6344TRPBF/IRLML6344TRPBFCT-ND/2538168" H 10100 2625 60  0001 C CNN "PurchasingLinks"
+	1    9800 2450
+	1    0    0    -1
+$EndComp
+Wire Wire Line
+	9900 1900 9900 2250
 $EndSCHEMATC

Commit message: more partsgit add *
Parts:
- added U?: RFTRANS434MHZ, rocketry:RFTRANS434MHZ, symbol RFTRANS434MHZ
Changed lines of the file:
@@
 Wire Wire Line
 	9900 1900 9900 2250
+$Comp
+L RFTRANS434MHZ U?
+U 1 1 5AD03B3C
+P 11800 3600
+F 0 "U?" H 11800 3200 60  0000 C CNN
+F 1 "RFTRANS434MHZ" H 11800 3800 60  0000 C CNN
+F 2 "rocketry:RFTRANS434MHZ" H 11700 3100 60  0001 C CNN
+F 3 "" H 11800 3200 60  0001 C CNN
+F 4 "https://www.sparkfun.com/products/10534" H 12150 3050 60  0001 C CNN "PurchasingLinks"
+	1    11800 3600
+	1    0    0    -1
+$EndComp
 $EndSCHEMATC

Commit message: added new accelerometer
Parts:
- added U?: ADX377, rocketry:ADXL377, symbol ADX377
Changed lines of the file:
@@
+	1    0    0    -1
+$EndComp
+$Comp
+L ADX377 U?
+U 1 1 5AD0D49E
+P 8750 4050
+F 0 "U?" H 8250 4800 60  0000 C CNN
+F 1 "ADX377" H 8300 3200 60  0000 C CNN
+F 2 "rocketry:ADXL377" H 8750 4450 60  0001 C CNN
+F 3 "" H 8750 4450 60  0001 C CNN
+F 4 "https://www.digikey.com/product-detail/en/analog-devices-inc/ADXL377BCPZ-RL7/ADXL377BCPZ-RL7CT-ND/3678489" H 8500 4900 60  0001 C CNN "PurchasingLinks"
+	1    8750 4050
 	1    0    0    -1
 $EndComp
