File: phoenix/phoenix.sch (KiCad schematic (older format))
At the start: 30 parts, among them J1 Ultrafit_2, J2 Micro_SD_Card_Det, P1 CONN_02X03, Q1 IRLML6344, U1 ATMEGA328P-AU, U3 MMA8451QT, U4 L6932D1.2, Y1 Crystal_SMD

Commit message: more components
Parts:
- added C? (x3): C_1000pF, footprints:C_0805_OEM, symbol C_1000pF
Connections:
- net GND: now also C?.2, C?.2
- net TX: now reaches U1.31 ((PCINT17/TXD)PD1)
- net TX: now also U?.2 (DATA)
- net at U?.16 (ZOUT): now also C?.1
- net at U?.4 (YOUT): now also C?.1
- net at U?.5 (XOUT): now also C?.1
- no-connect marks 27 -> 26
Changed lines of the file:
@@
 	16950 6500 16950 6350
 Wire Wire Line
-	18150 1300 18150 1600
-Wire Wire Line
-	18000 1500 18300 1500
+	18150 1300 18150 1500
+Wire Wire Line
+	18150 1500 18150 1600
+Wire Wire Line
+	18000 1500 18150 1500
+Wire Wire Line
+	18150 1500 18300 1500
 Wire Wire Line
 	18150 1600 18300 1600
@@
 	18300 3600 18200 3600
 Wire Wire Line
-	18200 3600 18200 3950
+	18200 3600 18200 3700
+Wire Wire Line
+	18200 3700 18200 3800
+Wire Wire Line
+	18200 3800 18200 3950
 Wire Wire Line
 	18300 3700 18200 3700
@@
 Connection ~ 18200 3800
 Wire Wire Line
-	20200 2950 20650 2950
+	20200 2950 20500 2950
+Wire Wire Line
+	20500 2950 20650 2950
 Wire Wire Line
 	20500 2900 20500 2950
@@
 	10200 5900 10550 5900
 Wire Wire Line
-	12200 2300 12200 2400
+	12200 2300 12200 2350
+Wire Wire Line
+	12200 2350 12200 2400
 Connection ~ 12200 2350
 Wire Wire Line
 	12200 2350 12650 2350
 Wire Wire Line
-	14850 2150 14850 2450
+	14850 2150 14850 2250
+Wire Wire Line
+	14850 2250 14850 2350
+Wire Wire Line
+	14850 2350 14850 2450
 Connection ~ 14850 2250
 Connection ~ 14850 2350
@@
 SEPERATE
 Wire Wire Line
-	20200 3800 20550 3800
+	20200 3800 20350 3800
+Wire Wire Line
+	20350 3800 20550 3800
 $Comp
 L R_10k R8
@@
 $EndComp
 Wire Wire Line
-	21750 2000 22050 2000
+	21750 2000 21900 2000
+Wire Wire Line
+	21900 2000 22050 2000
 Connection ~ 21400 2000
 Wire Wire Line
-	21300 2000 21550 2000
+	21300 2000 21400 2000
+Wire Wire Line
+	21400 2000 21550 2000
 Text Label 21300 2000 2    60   ~ 0
 PB6
@@
 	21650 1750 21950 1750
 Wire Wire Line
-	21650 2150 21650 2400
-Wire Wire Line
-	21400 2300 21900 2300
+	21650 2150 21650 2300
+Wire Wire Line
+	21650 2300 21650 2400
+Wire Wire Line
+	21400 2300 21650 2300
+Wire Wire Line
+	21650 2300 21900 2300
 Connection ~ 21650 2300
 Wire Wire Line
@@
 NoConn ~ 20200 3600
 NoConn ~ 20200 3500
-NoConn ~ 20200 3200
 NoConn ~ 20200 3100
 NoConn ~ 20200 2650
@@
 3.3V
 Wire Wire Line
-	10200 5200 10200 5600
+	10200 5200 10200 5450
+Wire Wire Line
+	10200 5450 10200 5600
 Wire Wire Line
 	10200 5200 10150 5200
@@
 Text Label 12100 3800 0    60   ~ 0
 3.3V
+$Comp
+L C_1000pF C?
+U 1 1 5AD2AF61
+P 9350 3850
+F 0 "C?" H 9375 3950 50  0000 L CNN
+F 1 "C_1000pF" H 9200 3850 50  0000 L CNN
+F 2 "footprints:C_0805_OEM" H 9300 3500 50  0001 C CNN
+F 3 "" H 9050 4100 50  0001 C CNN
+F 4 "CAP CER 1000pF 50V X7R 0805" H 9875 4450 60  0001 C CNN "Description"
+F 5 "1276-6843-1-ND " H 9350 3400 60  0001 C CNN "MPN"
+F 6 "Digi-Key" H 9350 3300 60  0001 C CNN "MFN"
+F 7 "Value" H 9350 3850 60  0001 C CNN "Package"
+F 8 "https://www.digikey.com/product-detail/en/samsung-electro-mechanics/CL21B102KB6WPNC/1276-6843-1-ND/5961702" H 9775 4350 60  0001 C CNN "PurchasingLink"
+	1    9350 3850
+	1    0    0    -1
+$EndComp
+$Comp
+L C_1000pF C?
+U 1 1 5AD2B025
+P 9650 3750
+F 0 "C?" H 9675 3850 50  0000 L CNN
+F 1 "C_1000pF" H 9675 3650 50  0000 L CNN
+F 2 "footprints:C_0805_OEM" H 9600 3400 50  0001 C CNN
+F 3 "" H 9350 4000 50  0001 C CNN
+F 4 "CAP CER 1000pF 50V X7R 0805" H 10175 4350 60  0001 C CNN "Description"
+F 5 "1276-6843-1-ND " H 9650 3300 60  0001 C CNN "MPN"
+F 6 "Digi-Key" H 9650 3200 60  0001 C CNN "MFN"
+F 7 "Value" H 9650 3750 60  0001 C CNN "Package"
+F 8 "https://www.digikey.com/product-detail/en/samsung-electro-mechanics/CL21B102KB6WPNC/1276-6843-1-ND/5961702" H 10075 4250 60  0001 C CNN "PurchasingLink"
+	1    9650 3750
+	1    0    0    -1
+$EndComp
+Text Label 9100 5100 3    60   ~ 0
+GND
+Wire Wire Line
+	8950 3700 9350 3700
+Text Label 9350 4000 3    60   ~ 0
+GND
+Text Label 9650 3900 3    60   ~ 0
+GND
+Wire Wire Line
+	8950 3600 9650 3600
+$Comp
+L C_1000pF C?
+U 1 1 5AD2B10B
+P 9050 4950
+F 0 "C?" H 9075 5050 50  0000 L CNN
+F 1 "C_1000pF" H 9075 4850 50  0000 L CNN
+F 2 "footprints:C_0805_OEM" H 9000 4600 50  0001 C CNN
+F 3 "" H 8750 5200 50  0001 C CNN
+F 4 "CAP CER 1000pF 50V X7R 0805" H 9575 5550 60  0001 C CNN "Description"
+F 5 "1276-6843-1-ND " H 9050 4500 60  0001 C CNN "MPN"
+F 6 "Digi-Key" H 9050 4400 60  0001 C CNN "MFN"
+F 7 "Value" H 9050 4950 60  0001 C CNN "Package"
+F 8 "https://www.digikey.com/product-detail/en/samsung-electro-mechanics/CL21B102KB6WPNC/1276-6843-1-ND/5961702" H 9475 5450 60  0001 C CNN "PurchasingLink"
+	1    9050 4950
+	1    0    0    -1
+$EndComp
+Wire Wire Line
+	8950 4800 9050 4800
+Text Label 20200 3200 0    60   ~ 0
+TX
+Text Label 12100 3700 0    60   ~ 0
+TX
 $EndSCHEMATC

Commit message: Draft layout
Added:
-changes to layout
-drafted tracing
-modified some footprints
-added 3d-file for micro-sd-card slot
Parts:
- gave numbers to parts that had none: 5
Connections:
- net GND: now also C8.2
- net PLED1: now also U1.2 ((PCINT20/XCK/T0)PD4); no longer U1.23 ((PCINT8/ADC0)PC0)
- net PLED2: now also U1.9 ((PCINT21/OC0B/T1)PD5); no longer U1.24 ((PCINT9/ADC1)PC1)
- net PLED3: now also U1.10 ((PCINT22/OC0A/AIN0)PD6); no longer U1.25 ((PCINT10/ADC2)PC2)
- net ZOUT: now reaches C8.1, U2.16 (ZOUT)
- net ZOUT: now also U1.25 ((PCINT10/ADC2)PC2)
- net YOUT: now reaches C10.1, U2.4 (YOUT)
- net YOUT: now also U1.23 ((PCINT8/ADC0)PC0)
- net XOUT: now reaches C9.1, U2.5 (XOUT)
- net XOUT: now also U1.24 ((PCINT9/ADC1)PC1)
- no-connect marks 26 -> 25
Changed lines of the file:
@@
 EESchema Schematic File Version 2
-LIBS:power
-LIBS:device
-LIBS:switches
-LIBS:relays
-LIBS:motors
-LIBS:transistors
-LIBS:conn
-LIBS:linear
-LIBS:regul
-LIBS:74xx
-LIBS:cmos4000
-LIBS:adc-dac
-LIBS:memory
-LIBS:xilinx
-LIBS:microcontrollers
-LIBS:dsp
-LIBS:microchip
-LIBS:analog_switches
-LIBS:motorola
-LIBS:texas
-LIBS:intel
-LIBS:audio
-LIBS:interface
-LIBS:digital-audio
-LIBS:philips
-LIBS:display
-LIBS:cypress
-LIBS:siliconi
-LIBS:opto
-LIBS:atmel
-LIBS:contrib
-LIBS:valves
 LIBS:rocketry
 LIBS:phoenix-cache
@@
 Text Label 16100 5050 1    60   ~ 0
 PLED3
-Text Label 20200 2350 0    60   ~ 0
+Text Label 20200 3500 0    60   ~ 0
 PLED1
-Text Label 20200 2450 0    60   ~ 0
+Text Label 20200 3600 0    60   ~ 0
 PLED2
-Text Label 20200 2550 0    60   ~ 0
+Text Label 20200 3700 0    60   ~ 0
 PLED3
 Text Notes 15100 4550 0    79   ~ 0
@@
 	16950 6500 16950 6350
 Wire Wire Line
-	18150 1300 18150 1500
-Wire Wire Line
-	18150 1500 18150 1600
-Wire Wire Line
-	18000 1500 18150 1500
-Wire Wire Line
-	18150 1500 18300 1500
+	18150 1300 18150 1600
+Wire Wire Line
+	18000 1500 18300 1500
 Wire Wire Line
 	18150 1600 18300 1600
@@
 	18300 3600 18200 3600
 Wire Wire Line
-	18200 3600 18200 3700
-Wire Wire Line
-	18200 3700 18200 3800
-Wire Wire Line
-	18200 3800 18200 3950
+	18200 3600 18200 3950
 Wire Wire Line
 	18300 3700 18200 3700
@@
 Connection ~ 18200 3800
 Wire Wire Line
-	20200 2950 20500 2950
-Wire Wire Line
-	20500 2950 20650 2950
+	20200 2950 20650 2950
 Wire Wire Line
 	20500 2900 20500 2950
@@
 	10200 5900 10550 5900
 Wire Wire Line
-	12200 2300 12200 2350
-Wire Wire Line
-	12200 2350 12200 2400
+	12200 2300 12200 2400
 Connection ~ 12200 2350
 Wire Wire Line
 	12200 2350 12650 2350
 Wire Wire Line
-	14850 2150 14850 2250
-Wire Wire Line
-	14850 2250 14850 2350
-Wire Wire Line
-	14850 2350 14850 2450
+	14850 2150 14850 2450
 Connection ~ 14850 2250
 Connection ~ 14850 2350
@@
 SEPERATE
 Wire Wire Line
-	20200 3800 20350 3800
-Wire Wire Line
-	20350 3800 20550 3800
+	20200 3800 20550 3800
 $Comp
 L R_10k R8
@@
 $EndComp
 Wire Wire Line
-	21750 2000 21900 2000
-Wire Wire Line
-	21900 2000 22050 2000
+	21750 2000 22050 2000
 Connection ~ 21400 2000
 Wire Wire Line
-	21300 2000 21400 2000
-Wire Wire Line
-	21400 2000 21550 2000
+	21300 2000 21550 2000
 Text Label 21300 2000 2    60   ~ 0
 PB6
@@
 	21650 1750 21950 1750
 Wire Wire Line
-	21650 2150 21650 2300
-Wire Wire Line
-	21650 2300 21650 2400
-Wire Wire Line
-	21400 2300 21650 2300
-Wire Wire Line
-	21650 2300 21900 2300
+	21650 2150 21650 2400
+Wire Wire Line
+	21400 2300 21900 2300
 Connection ~ 21650 2300
 Wire Wire Line
@@
 NoConn ~ 18300 2950
 NoConn ~ 18300 2850
-NoConn ~ 20200 3700
-NoConn ~ 20200 3600
-NoConn ~ 20200 3500
 NoConn ~ 20200 3100
 NoConn ~ 20200 2650
@@
 3.3V
 Wire Wire Line
-	10200 5200 10200 5450
-Wire Wire Line
-	10200 5450 10200 5600
+	10200 5200 10200 5600
 Wire Wire Line
 	10200 5200 10150 5200
@@
 	9900 1900 9900 2250
 $Comp
-L RFTRANS434MHZ U?
+L RFTRANS434MHZ U5
 U 1 1 5AD03B3C
 P 11800 3600
-F 0 "U?" H 11800 3200 60  0000 C CNN
+F 0 "U5" H 11800 3200 60  0000 C CNN
 F 1 "RFTRANS434MHZ" H 11800 3800 60  0000 C CNN
 F 2 "rocketry:RFTRANS434MHZ" H 11700 3100 60  0001 C CNN
@@
 $EndComp
 $Comp
-L ADX377 U?
+L ADX377 U2
 U 1 1 5AD0D49E
 P 8750 4050
-F 0 "U?" H 8250 4800 60  0000 C CNN
+F 0 "U2" H 8250 4800 60  0000 C CNN
 F 1 "ADX377" H 8300 3200 60  0000 C CNN
 F 2 "rocketry:ADXL377" H 8750 4450 60  0001 C CNN
@@
 3.3V
 $Comp
-L C_1000pF C?
+L C_1000pF C9
 U 1 1 5AD2AF61
 P 9350 3850
-F 0 "C?" H 9375 3950 50  0000 L CNN
+F 0 "C9" H 9375 3950 50  0000 L CNN
 F 1 "C_1000pF" H 9200 3850 50  0000 L CNN
 F 2 "footprints:C_0805_OEM" H 9300 3500 50  0001 C CNN
@@
 $EndComp
 $Comp
-L C_1000pF C?
+L C_1000pF C10
 U 1 1 5AD2B025
 P 9650 3750
-F 0 "C?" H 9675 3850 50  0000 L CNN
+F 0 "C10" H 9675 3850 50  0000 L CNN
 F 1 "C_1000pF" H 9675 3650 50  0000 L CNN
 F 2 "footprints:C_0805_OEM" H 9600 3400 50  0001 C CNN
@@
 	1    0    0    -1
 $EndComp
-Text Label 9100 5100 3    60   ~ 0
+Text Label 9050 5100 3    60   ~ 0
 GND
 Wire Wire Line
@@
 	8950 3600 9650 3600
 $Comp
-L C_1000pF C?
+L C_1000pF C8
 U 1 1 5AD2B10B
 P 9050 4950
-F 0 "C?" H 9075 5050 50  0000 L CNN
+F 0 "C8" H 9075 5050 50  0000 L CNN
 F 1 "C_1000pF" H 9075 4850 50  0000 L CNN
 F 2 "footprints:C_0805_OEM" H 9000 4600 50  0001 C CNN
@@
 Text Label 12100 3700 0    60   ~ 0
 TX
+NoConn ~ 8950 3400
+NoConn ~ 12100 3900
+Text Label 9650 3600 0    60   ~ 0
+YOUT
+Text Label 9350 3700 0    60   ~ 0
+XOUT
+Text Label 9050 4800 0    60   ~ 0
+ZOUT
+Text Label 20200 2450 0    60   ~ 0
+XOUT
+Text Label 20200 2350 0    60   ~ 0
+YOUT
+Text Label 20200 2550 0    60   ~ 0
+ZOUT
 $EndSCHEMATC

Commit message: update to kicad 5
Parts:
- BT1: symbol Battery_Cell -> phoenix-rescue:Battery_Cell
- C1, C2: symbol C_0.1uF -> rocketry:C_0.1uF
- C10, C8, C9: symbol C_1000pF -> rocketry:C_1000pF
- C3, C4: symbol C_10uF -> rocketry:C_10uF
- C5: symbol C_100pF -> rocketry:C_100pF
- C6, C7: symbol C_30pF -> rocketry:C_30pF
- D1, D2, D3: symbol LED_0805 -> rocketry:LED_0805
- J1: symbol Ultrafit_2 -> rocketry:Ultrafit_2
- J2: symbol Micro_SD_Card_Det -> phoenix-rescue:Micro_SD_Card_Det
- P1: symbol CONN_02X03 -> rocketry:CONN_02X03
- Q1: symbol IRLML6344 -> rocketry:IRLML6344
- R1, R8, R9: symbol R_10k -> rocketry:R_10k
- R2, R3: symbol 5K -> rocketry:5K
- R4, R5, R6: symbol R_200 -> rocketry:R_200
- R7: symbol R_100 -> rocketry:R_100
- U1: symbol ATMEGA328P-AU -> phoenix-rescue:ATMEGA328P-AU
- U2: symbol ADX377 -> rocketry:ADX377
- U3: symbol MMA8451QT -> rocketry:MMA8451QT
- U4: symbol L6932D1.2 -> rocketry:L6932D1.2
- U5: symbol RFTRANS434MHZ -> rocketry:RFTRANS434MHZ
- Y1: symbol Crystal_SMD -> rocketry:Crystal_SMD
Changed lines of the file:
@@
-EESchema Schematic File Version 2
-LIBS:rocketry
+EESchema Schematic File Version 4
 LIBS:phoenix-cache
-EELAYER 25 0
+EELAYER 26 0
 EELAYER END
 $Descr A2 23386 16535
@@
 $EndDescr
 $Comp
-L Battery_Cell BT1
+L phoenix-rescue:Battery_Cell BT1
 U 1 1 5ABA39D7
 P 17700 6450
@@
 $EndComp
 $Comp
-L Micro_SD_Card_Det J2
+L phoenix-rescue:Micro_SD_Card_Det J2
 U 1 1 5ABA3E17
 P 19850 5750
@@
 $EndComp
 $Comp
-L ATMEGA328P-AU U1
+L phoenix-rescue:ATMEGA328P-AU U1
 U 1 1 5A8B2ED4
 P 19200 2600
@@
 SCK
 $Comp
-L +3.3V #PWR01
+L power:+3.3V #PWR01
 U 1 1 5ABBE98B
 P 16550 6500
@@
 GND
 $Comp
-L GND #PWR02
+L power:GND #PWR02
 U 1 1 5ABBEBF9
 P 16950 6500
@@
 $EndComp
 $Comp
-L PWR_FLAG #FLG03
+L power:PWR_FLAG #FLG03
 U 1 1 5ABBECDC
 P 15700 6450
@@
 $EndComp
 $Comp
-L PWR_FLAG #FLG04
+L power:PWR_FLAG #FLG04
 U 1 1 5ABBED0C
 P 16100 6450
@@
 $EndComp
 $Comp
-L PWR_FLAG #FLG05
+L power:PWR_FLAG #FLG05
 U 1 1 5ABBED35
 P 15300 6450
@@
 $EndComp
 $Comp
-L +3.3V #PWR06
+L power:+3.3V #PWR06
 U 1 1 5ABBED86
 P 15700 6450
@@
 $EndComp
 $Comp
-L GND #PWR07
+L power:GND #PWR07
 U 1 1 5ABBEDAF
 P 16100 6450
@@
 $EndComp
 $Comp
-L R_100 R7
+L rocketry:R_100 R7
 U 1 1 5ABBF03F
 P 18000 1650
@@
 $EndComp
 $Comp
-L C_100pF C5
+L rocketry:C_100pF C5
 U 1 1 5ABBF093
 P 18000 2000
@@
 NoConn ~ 18300 2100
 $Comp
-L GND #PWR08
+L power:GND #PWR08
 U 1 1 5ABBF3B0
 P 18000 2150
@@
 $EndComp
 $Comp
-L +BATT #PWR09
+L power:+BATT #PWR09
 U 1 1 5ABBF3D1
 P 15300 6450
@@
 $EndComp
 $Comp
-L GND #PWR010
+L power:GND #PWR010
 U 1 1 5ABBF579
 P 18200 3950
@@
 $EndComp
 $Comp
-L CONN_02X03 P1
+L rocketry:CONN_02X03 P1
 U 1 1 5ABBF86C
 P 17150 5600
@@
 RESET
 $Comp
-L R_10k R9
+L rocketry:R_10k R9
 U 1 1 5ABBFB31
 P 20500 2750
@@
 MOSI
 $Comp
-L GND #PWR011
+L power:GND #PWR011
 U 1 1 5ABBFD0B
 P 17450 5750
@@
 NoConn ~ 18950 6050
 $Comp
-L GND #PWR012
+L power:GND #PWR012
 U 1 1 5ABBFDCC
 P 18600 5950
@@
 $EndComp
 $Comp
-L LED_0805 D2
+L rocketry:LED_0805 D2
 U 1 1 5ABC351F
 P 15750 5200
@@
 $EndComp
 $Comp
-L R_200 R5
+L rocketry:R_200 R5
 U 1 1 5ABC3594
 P 15750 5650
@@
 $EndComp
 $Comp
-L GND #PWR013
+L power:GND #PWR013
 U 1 1 5ABC363D
 P 15750 5800
@@
 $EndComp
 $Comp
-L LED_0805 D3
+L rocketry:LED_0805 D3
 U 1 1 5ABC379F
 P 16100 5200
@@
 $EndComp
 $Comp
-L R_200 R6
+L rocketry:R_200 R6
 U 1 1 5ABC37A9
 P 16100 5650
@@
 $EndComp
 $Comp
-L GND #PWR014
+L power:GND #PWR014
 U 1 1 5ABC37AF
 P 16100 5800
@@
 $EndComp
 $Comp
-L LED_0805 D1
+L rocketry:LED_0805 D1
 U 1 1 5ABC380C
 P 15400 5200
@@
 $EndComp
 $Comp
-L R_200 R4
+L rocketry:R_200 R4
 U 1 1 5ABC3816
 P 15400 5650
@@
 $EndComp
 $Comp
-L GND #PWR015
+L power:GND #PWR015
 U 1 1 5ABC381C
 P 15400 5800
@@
 Micro SD-Card Reader
 $Comp
-L Ultrafit_2 J1
+L rocketry:Ultrafit_2 J1
 U 1 1 5ABC44C9
 P 9550 1850
@@
 $EndComp
 $Comp
-L MMA8451QT U3
+L rocketry:MMA8451QT U3
 U 1 1 5AC3B52F
 P 10550 5300
@@
 NoConn ~ 10550 6000
 $Comp
-L C_0.1uF C1
+L rocketry:C_0.1uF C1
 U 1 1 5AC40F79
 P 9800 5700
@@
 GND
 $Comp
-L R_10k R1
+L rocketry:R_10k R1
 U 1 1 5AC414DA
 P 10200 5750
@@
 $EndComp
 $Comp
-L C_0.1uF C2
+L rocketry:C_0.1uF C2
 U 1 1 5AC416EE
 P 9300 5700
@@
 SCL
 $Comp
-L L6932D1.2 U4
+L rocketry:L6932D1.2 U4
 U 1 1 5AC43804
 P 12650 2150
@@
 $EndComp
 $Comp
-L C_10uF C4
+L rocketry:C_10uF C4
 U 1 1 5AC43E21
 P 11800 2250
@@
 VIN
 $Comp
-L 5K R3
+L rocketry:5K R3
 U 1 1 5AC3FF90
 P 12200 2550
@@
 $EndComp
 $Comp
-L 5K R2
+L rocketry:5K R2
 U 1 1 5AC404C1
 P 12200 2150
@@
 VIN
 $Comp
-L C_10uF C3
+L rocketry:C_10uF C3
 U 1 1 5AC40A51
 P 11400 2250
@@
 	16950 6500 16950 6350
 Wire Wire Line
-	18150 1300 18150 1600
-Wire Wire Line
-	18000 1500 18300 1500
+	18150 1300 18150 1500
+Wire Wire Line
+	18000 1500 18150 1500
 Wire Wire Line
 	18150 1600 18300 1600
@@
 	18300 3600 18200 3600
 Wire Wire Line
-	18200 3600 18200 3950
+	18200 3600 18200 3700
 Wire Wire Line
 	18300 3700 18200 3700
@@
 Connection ~ 18200 3800
 Wire Wire Line
-	20200 2950 20650 2950
+	20200 2950 20500 2950
 Wire Wire Line
 	20500 2900 20500 2950
@@
 	10200 5900 10550 5900
 Wire Wire Line
-	12200 2300 12200 2400
+	12200 2300 12200 2350
 Connection ~ 12200 2350
 Wire Wire Line
 	12200 2350 12650 2350
 Wire Wire Line
-	14850 2150 14850 2450
+	14850 2150 14850 2250
 Connection ~ 14850 2250
 Connection ~ 14850 2350
@@
 SEPERATE
 Wire Wire Line
-	20200 3800 20550 3800
-$Comp
-L R_10k R8
+	20200 3800 20350 3800
+$Comp
+L rocketry:R_10k R8
 U 1 1 5AC43E0B
 P 20350 3950
@@
 N-Channel Transistor\n
 $Comp
-L Crystal_SMD Y1
+L rocketry:Crystal_SMD Y1
 U 1 1 5ACEF03D
 P 21650 2000
@@
 GND
 $Comp
-L C_30pF C6
+L rocketry:C_30pF C6
 U 1 1 5ACF00B7
 P 21400 2150
@@
 $EndComp
 $Comp
-L C_30pF C7
+L rocketry:C_30pF C7
 U 1 1 5ACF0160
 P 21900 2150
@@
 $EndComp
 Wire Wire Line
-	21750 2000 22050 2000
+	21750 2000 21900 2000
 Connection ~ 21400 2000
 Wire Wire Line
-	21300 2000 21550 2000
+	21300 2000 21400 2000
 Text Label 21300 2000 2    60   ~ 0
 PB6
@@
 	21650 1750 21950 1750
 Wire Wire Line
-	21650 2150 21650 2400
-Wire Wire Line
-	21400 2300 21900 2300
+	21650 2150 21650 2300
+Wire Wire Line
+	21400 2300 21650 2300
 Connection ~ 21650 2300
 Wire Wire Line
@@
 3.3V
 Wire Wire Line
-	10200 5200 10200 5600
+	10200 5200 10200 5450
 Wire Wire Line
 	10200 5200 10150 5200
@@
 NoConn ~ 20650 6250
 $Comp
-L IRLML6344 Q1
+L rocketry:IRLML6344 Q1
 U 1 1 5ACFF80D
 P 9800 2450
@@
 	9900 1900 9900 2250
 $Comp
-L RFTRANS434MHZ U5
+L rocketry:RFTRANS434MHZ U5
 U 1 1 5AD03B3C
 P 11800 3600
@@
 $EndComp
 $Comp
-L ADX377 U2
+L rocketry:ADX377 U2
 U 1 1 5AD0D49E
 P 8750 4050
@@
 3.3V
 $Comp
-L C_1000pF C9
+L rocketry:C_1000pF C9
 U 1 1 5AD2AF61
 P 9350 3850
@@
 $EndComp
 $Comp
-L C_1000pF C10
+L rocketry:C_1000pF C10
 U 1 1 5AD2B025
 P 9650 3750
@@
 	8950 3600 9650 3600
 $Comp
-L C_1000pF C8
+L rocketry:C_1000pF C8
 U 1 1 5AD2B10B
 P 9050 4950
@@
 Text Label 20200 2550 0    60   ~ 0
 ZOUT
+Wire Wire Line
+	18150 1500 18150 1600
+Wire Wire Line
+	18150 1500 18300 1500
+Wire Wire Line
+	18200 3700 18200 3800
+Wire Wire Line
+	18200 3800 18200 3950
+Wire Wire Line
+	20500 2950 20650 2950
+Wire Wire Line
+	12200 2350 12200 2400
+Wire Wire Line
+	14850 2250 14850 2350
+Wire Wire Line
+	14850 2350 14850 2450
+Wire Wire Line
+	20350 3800 20550 3800
+Wire Wire Line
+	21400 2000 21550 2000
+Wire Wire Line
+	21900 2000 22050 2000
+Wire Wire Line
+	21650 2300 21650 2400
+Wire Wire Line
+	21650 2300 21900 2300
+Wire Wire Line
+	10200 5450 10200 5600
 $EndSCHEMATC
