File: phoenix/phoenix.kicad_pcb (KiCad board)
At the start: 2 copper layers, 65 x 22.6 mm, 35 parts, among them J1 Ultrafit_2, J2 Micro_SD_Card_Det, J4 Ultrafit_2, J5 Ultrafit_2, P1 CONN_02X03, Q1 IRLML6344, U1 ATMEGA328P-AU, U2 ADX377, U3 MMA8451QT, U4 L6932D1.2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

Commit message: cleanup
Parts:
- moved Q1 1.49 mm to (163.0, 70.4)
Routing:
- net GND: track 75.6 -> 68.5 mm, vias 18 -> 17
- net /SEPERATE: track 34.7 -> 31.4 mm
Changed lines of the file:
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@@
   (general
     (links 96)
-    (no_connects 0)
+    (no_connects 4)
     (area 106.604999 53.518999 171.779001 76.275001)
     (thickness 1.6)
     (drawings 12)
-    (tracks 459)
+    (tracks 450)
     (zones 0)
     (modules 35)
@@
   )
   (module footprints:Ultrafit_2 (layer F.Cu)
+    (at 167.95 71.12)
+    (fp_text reference J1 (at 5.08 5.08) (layer F.SilkS)
+      (effects (font (size 1 1) (thickness 0.15)))
+    )
+    (fp_text value Ultrafit_2 (at 4.572 0.508 90) (layer F.Fab) hide
+      (effects (font (size 1 1) (thickness 0.15)))
+    )
+    (fp_line (start -5.588 -2.032) (end -2.54 -2.032) (layer F.Fab) (width 0.15))
+    (fp_line (start -2.54 -2.032) (end -2.54 5.588) (layer F.Fab) (width 0.15))
+    (fp_line (start -2.54 5.588) (end -5.588 5.588) (layer F.Fab) (width 0.15))
+    (fp_line (start -5.588 5.588) (end -5.588 -2.032) (layer F.Fab) (width 0.15))
+    (fp_text user "6.55mm Clearance" (at -4.07 1.75 90) (layer F.Fab)
+      (effects (font (size 0.5 0.5) (thickness 0.08)))
+    )
+    (fp_line (start -2.42 -2.15) (end -5.73 -2.15) (layer F.SilkS) (width 0.15))
+    (fp_line (start -5.73 -2.15) (end -5.73 5.65) (layer F.SilkS) (width 0.15))
+    (fp_line (start -5.73 5.65) (end -2.42 5.65) (layer F.SilkS) (width 0.15))
+    (fp_line (start -2.42 5.65) (end 3.302 5.65) (layer F.SilkS) (width 0.15))
+    (fp_line (start -2.42 -2.15) (end 3.302 -2.15) (layer F.SilkS) (width 0.15))
+    (fp_line (start -2.42 5.65) (end -2.42 -2.15) (layer F.SilkS) (width 0.15))
+    (fp_line (start 3.302 5.65) (end 3.302 -2.15) (layer F.SilkS) (width 0.15))
+    (pad 2 thru_hole circle (at 0 0) (size 1.397 1.397) (drill 1.02) (layers *.Cu *.Mask)
+      (net 21 "Net-(J1-Pad2)"))
+    (pad 1 thru_hole circle (at 0 3.5) (size 1.397 1.397) (drill 1.02) (layers *.Cu *.Mask)
+      (net 8 +3V3))
+    (pad "" smd circle (at 2.23 1.75) (size 1.981 1.981) (layers Dwgs.User))
+  )
+  (module footprints:Ultrafit_2 (layer F.Cu)
     (at 124.615 75.001 90)
     (fp_text reference J5 (at -0.183 1.6738 180) (layer F.SilkS)
@@
       (rotate (xyz 0 0 0))
     )
-  )
-  (module footprints:Ultrafit_2 (layer F.Cu)
-    (at 167.95 71.12)
-    (fp_text reference J1 (at 5.08 5.08) (layer F.SilkS)
-      (effects (font (size 1 1) (thickness 0.15)))
-    )
-    (fp_text value Ultrafit_2 (at 4.572 0.508 90) (layer F.Fab) hide
-      (effects (font (size 1 1) (thickness 0.15)))
-    )
-    (fp_line (start -5.588 -2.032) (end -2.54 -2.032) (layer F.Fab) (width 0.15))
-    (fp_line (start -2.54 -2.032) (end -2.54 5.588) (layer F.Fab) (width 0.15))
-    (fp_line (start -2.54 5.588) (end -5.588 5.588) (layer F.Fab) (width 0.15))
-    (fp_line (start -5.588 5.588) (end -5.588 -2.032) (layer F.Fab) (width 0.15))
-    (fp_text user "6.55mm Clearance" (at -4.07 1.75 90) (layer F.Fab)
-      (effects (font (size 0.5 0.5) (thickness 0.08)))
-    )
-    (fp_line (start -2.42 -2.15) (end -5.73 -2.15) (layer F.SilkS) (width 0.15))
-    (fp_line (start -5.73 -2.15) (end -5.73 5.65) (layer F.SilkS) (width 0.15))
-    (fp_line (start -5.73 5.65) (end -2.42 5.65) (layer F.SilkS) (width 0.15))
-    (fp_line (start -2.42 5.65) (end 3.302 5.65) (layer F.SilkS) (width 0.15))
-    (fp_line (start -2.42 -2.15) (end 3.302 -2.15) (layer F.SilkS) (width 0.15))
-    (fp_line (start -2.42 5.65) (end -2.42 -2.15) (layer F.SilkS) (width 0.15))
-    (fp_line (start 3.302 5.65) (end 3.302 -2.15) (layer F.SilkS) (width 0.15))
-    (pad 2 thru_hole circle (at 0 0) (size 1.397 1.397) (drill 1.02) (layers *.Cu *.Mask)
-      (net 21 "Net-(J1-Pad2)"))
-    (pad 1 thru_hole circle (at 0 3.5) (size 1.397 1.397) (drill 1.02) (layers *.Cu *.Mask)
-      (net 8 +3V3))
-    (pad "" smd circle (at 2.23 1.75) (size 1.981 1.981) (layers Dwgs.User))
   )
   (module Housings_QFP:TQFP-32_7x7mm_Pitch0.8mm (layer F.Cu)
@@
       (net 9 GND))
   )
-  (module rocketry:IRLML6344TRPBFCT-ND (layer F.Cu)
-    (at 162.88 71.89)
-    (fp_text reference Q1 (at 0.95 -1.151) (layer F.SilkS)
-      (effects (font (size 1 1) (thickness 0.15)))
-    )
-    (fp_text value IRLML6344 (at 2.14884 -3.92684) (layer F.Fab)
-      (effects (font (size 1 1) (thickness 0.15)))
-    )
-    (fp_line (start -0.45212 2.21996) (end 2.34696 2.21996) (layer F.SilkS) (width 0.15))
-    (fp_line (start 2.34696 -0.42164) (end 2.34696 2.21996) (layer F.SilkS) (width 0.15))
-    (fp_line (start -0.45 -0.4191) (end -0.45 2.2209) (layer F.SilkS) (width 0.15))
-    (fp_line (start -0.45 -0.4191) (end 2.35 -0.4191) (layer F.SilkS) (width 0.15))
-    (pad 1 smd rect (at 0 0) (size 0.802 0.972) (layers F.Cu F.Paste F.Mask)
-      (net 27 /SEPERATE))
-    (pad 3 smd rect (at 0.95 1.77) (size 0.802 0.972) (layers F.Cu F.Paste F.Mask)
-      (net 21 "Net-(J1-Pad2)"))
-    (pad 2 smd rect (at 1.9 0) (size 0.802 0.972) (layers F.Cu F.Paste F.Mask)
-      (net 9 GND))
-  )
   (module footprints:C_0805_OEM (layer F.Cu)
     (at 132.858 69.85 180)
@@
       (net 50 "Net-(U5-Pad4)"))
   )
+  (module rocketry:IRLML6344TRPBFCT-ND (layer F.Cu)
+    (at 163.0426 70.4088)
+    (fp_text reference Q1 (at 0.95 -1.151) (layer F.SilkS)
+      (effects (font (size 1 1) (thickness 0.15)))
+    )
+    (fp_text value IRLML6344 (at 2.14884 -3.92684) (layer F.Fab)
+      (effects (font (size 1 1) (thickness 0.15)))
+    )
+    (fp_line (start -0.45212 2.21996) (end 2.34696 2.21996) (layer F.SilkS) (width 0.15))
+    (fp_line (start 2.34696 -0.42164) (end 2.34696 2.21996) (layer F.SilkS) (width 0.15))
+    (fp_line (start -0.45 -0.4191) (end -0.45 2.2209) (layer F.SilkS) (width 0.15))
+    (fp_line (start -0.45 -0.4191) (end 2.35 -0.4191) (layer F.SilkS) (width 0.15))
+    (pad 2 smd rect (at 0 0) (size 0.802 0.972) (layers F.Cu F.Paste F.Mask)
+      (net 9 GND))
+    (pad 3 smd rect (at 0.95 1.77) (size 0.802 0.972) (layers F.Cu F.Paste F.Mask)
+      (net 21 "Net-(J1-Pad2)"))
+    (pad 1 smd rect (at 1.9 0) (size 0.802 0.972) (layers F.Cu F.Paste F.Mask)
+      (net 27 /SEPERATE))
+  )
   (dimension 64.998605 (width 0.3) (layer Dwgs.User)
     (gr_text "2.5590 in" (at 139.176758 46.822629 0.02238990879) (layer Dwgs.User)
@@
   (gr_line (start 171.704 53.594) (end 171.704 76.2) (layer Edge.Cuts) (width 0.15))
   (gr_line (start 106.68 53.594) (end 171.704 53.594) (layer Edge.Cuts) (width 0.15))
+  (segment (start 164.78 71.975) (end 164.78 71.89) (width 0.254) (layer F.Cu) (net 0))
+  (segment (start 162.88 71.975) (end 162.88 71.89) (width 0.254) (layer F.Cu) (net 0))
   (segment (start 140.716 57.658) (end 140.716 55.109078) (width 0.254) (layer F.Cu) (net 2))
   (segment (start 140.716 55.109078) (end 141.659577 54.165501) (width 0.254) (layer F.Cu) (net 2))
@@
   (segment (start 146.726321 64.454973) (end 146.774648 64.5033) (width 0.254) (layer F.Cu) (net 9))
   (segment (start 146.774648 64.5033) (end 147.2057 64.5033) (width 0.254) (layer F.Cu) (net 9))
-  (segment (start 164.78 71.89) (end 165.9683 71.89) (width 0.254) (layer F.Cu) (net 9))
-  (segment (start 165.9683 71.89) (end 165.9763 71.882) (width 0.254) (layer F.Cu) (net 9))
-  (via (at 165.9763 71.882) (size 0.6096) (drill 0.3048) (layers F.Cu B.Cu) (net 9))
-  (segment (start 160.02 74.61) (end 161.549922 74.61) (width 0.254) (layer F.Cu) (net 9))
-  (segment (start 161.549922 74.61) (end 163.529922 72.63) (width 0.254) (layer F.Cu) (net 9))
-  (segment (start 163.529922 72.63) (end 164.125 72.63) (width 0.254) (layer F.Cu) (net 9))
-  (segment (start 164.125 72.63) (end 164.78 71.975) (width 0.254) (layer F.Cu) (net 9))
-  (segment (start 164.78 71.975) (end 164.78 71.89) (width 0.254) (layer F.Cu) (net 9))
   (segment (start 155.432 74.93) (end 156.6164 74.93) (width 0.254) (layer F.Cu) (net 9))
   (segment (start 156.6164 74.93) (end 156.6291 74.9173) (width 0.254) (layer F.Cu) (net 9))
@@
   (segment (start 156.336999 67.858641) (end 156.336999 66.547999) (width 0.254) (layer F.Cu) (net 27))
   (via (at 155.321 65.532) (size 0.6096) (drill 0.3048) (layers F.Cu B.Cu) (net 27))
-  (segment (start 160.02 72.71) (end 162.145 72.71) (width 0.254) (layer F.Cu) (net 27))
-  (segment (start 162.145 72.71) (end 162.88 71.975) (width 0.254) (layer F.Cu) (net 27))
-  (segment (start 162.88 71.975) (end 162.88 71.89) (width 0.254) (layer F.Cu) (net 27))
   (segment (start 144.5768 74.406001) (end 145.3134 74.406001) (width 0.254) (layer F.Cu) (net 28))
   (segment (start 145.22 68.099) (end 145.22 67.57) (width 0.254) (layer F.Cu) (net 28))
