File: peregrine/flight_computer/flight_computer.kicad_pcb (KiCad board)
At the start: 2 copper layers, 34 parts, among them J1 Micro_SD_Card_Det, P1 CONN_02X03, U1 ATmega328PB-AU, U2 MIC5504-3.3YM5, U3 BMI088, U4 BMP388, U5 ICG-20660, U6 AT25SF041, U7 RFTRANS434MHZ, Y1 Crystal_SMD

Commit message: Updated
Parts:
- added J2: Conn_01x02_Male, rocketry:JST_90DEG_2PIN, B.Cu at (96.5, 92.3)
- AE1, J1, U7: moved to B.Cu
- moved U2 74.5 mm to (75.7, 96.5)
- moved C2 66.5 mm to (78.5, 96.5), turned to 270 degrees
- moved C1 66.0 mm to (72.8, 96.5), turned to 270 degrees
- moved D1 52.5 mm to (81.2, 79.3), turned to 0 degrees
- moved R3 50.1 mm to (84.8, 79.2), turned to 0 degrees
- moved AE1 45.8 mm to (86.1, 64.1)
- moved D2 41.1 mm to (71.0, 82.4)
- moved C4 37.3 mm to (72.2, 78.4), turned to 90 degrees
- moved D3 36.4 mm to (71.0, 90.7), turned to 270 degrees
- moved R4 35.5 mm to (71.7, 85.3), turned to 0 degrees
- moved R5 35.2 mm to (71.7, 87.8), turned to 0 degrees
- moved C13 34.4 mm to (79.1, 81.1), turned to 180 degrees
- moved P1 34.4 mm to (92.6, 65.0), turned to 90 degrees
- moved Y1 33.3 mm to (75.2, 78.3), turned to 180 degrees
- moved U7 32.7 mm to (72.3, 63.9), turned to 270 degrees
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Connections:
- C1 pad 1: +3V3 -> +BATT
- D2 pad 1: GND -> Net-(D2-Pad1)
- D2 pad 2: Net-(D2-Pad2) -> +3V3
- D3 pad 1: GND -> Net-(D3-Pad1)
- D3 pad 2: Net-(D3-Pad2) -> +3V3
- R4 pad 1: Net-(D2-Pad2) -> Net-(D2-Pad1)
- R5 pad 1: Net-(D3-Pad2) -> Net-(D3-Pad1)
- U2 pad 1: +3V3 -> +BATT
- U2 pad 3: +3V3 -> +BATT
Routing:
- net GND: track 0.00 -> 201.9 mm, vias 0 -> 21
- net +3V3: track 85.0 -> 162.3 mm, vias 4 -> 8
- net +BATT: track 0.00 -> 44.7 mm, vias 0 -> 1
- net /MOSI: track 42.2 -> 58.1 mm, vias 4 -> 5
- net /CS_FLASH: track 8.96 -> 21.5 mm, vias 0 -> 2
- net /CS_SD: track 0.00 -> 11.6 mm, vias 0 -> 1
- net /SCK: track 46.6 -> 57.3 mm
- net Net-(AE1-Pad1): track 0.00 -> 6.33 mm
- net /SCL: track 27.0 -> 22.2 mm, vias 3 -> 4
- net /MISO: track 56.3 -> 53.0 mm, vias 2 -> 3
- net /TXD: track 28.0 -> 30.0 mm, vias 2 -> 5
- net Net-(D3-Pad1): track 0.00 -> 1.93 mm
- net Net-(D2-Pad1): track 0.00 -> 1.93 mm
- net Net-(D3-Pad2): track 1.76 -> 0.00 mm
- net /LED_B: track 0.00 -> 1.73 mm
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- added copper zone on B.Cu, net GND
- added copper zone on F.Cu, net GND
Other:
- board outline added: 30 x 40 mm
- rule trace_min: 0.2 -> 0.16
- rule via_min_size: 0.4 -> 0.5

Commit message: Final rev?
Parts:
- added F1: Fuse, rocketry:Fuse_1210, F.Cu at (97.9, 95.5)
Connections:
- J2 pad 1: +BATT -> Net-(F1-Pad2)
Routing:
- net GND: track 201.9 -> 215.8 mm, vias 21 -> 71
- net +BATT: track 44.7 -> 38.8 mm, vias 1 -> 0
- net Net-(F1-Pad2): track 0.00 -> 3.50 mm, vias 0 -> 1
- net +3V3: track 162.3 -> 163.6 mm
- net /SCL: track 22.2 -> 23.1 mm
Other:
- net class Default: via_dia 0.8 -> 0.5; via_drill 0.4 -> 0.3

Commit message: Jesus help me
Parts:
- added G***: not_me, KiCad_Schematics:not_me, B.Cu at (93.6, 78.7)
- added G***: me, KiCad_Schematics:me, B.Cu at (74.8, 95.2)
- renumbered C13 to ←C13
Other:
- board text added: "//SCARY RF HERE KEEP OUT"
- board text added: "Peregrine, Rev 1 Solomon & Will"
